File: Common_Modules/Gyroscope/Gyroscope_breakout.kicad_pcb (KiCad board)
At the start: 2 copper layers, 30 x 22.9 mm, 5 parts, among them IC101 BMI088, J101 Conn_01x08, J102 Conn_01x08

Commit message: Restructured and reformatted to standards
There was an unneccessary folder that I got rid of, also updated the project so that it follows the standards set out in the Cerberus Github GUide
Parts:
- removed J102: Conn_01x08, Connector_PinHeader_2.54mm:PinHeader_1x08_P2.54mm_Vertical
- added e101: Conn_01x08, Gyroscope:PinHeader_1x08_P2.54mm_Vertical, F.Cu at (137.2, 86.9)
- C101, C102: footprint Capacitor_SMD:C_0201_0603Metric -> Gyroscope:C_0201_0603Metric
- IC101: footprint ERFSEDS_Footprints:16-LGA-(4.5x3) -> Gyroscope:16-LGA-(4.5x3)
- J101: footprint Connector_PinHeader_2.54mm:PinHeader_1x08_P2.54mm_Vertical -> Gyroscope:PinHeader_1x08_P2.54mm_Vertical
