File: Accelerometer_Breakout/Breakout_Board/Accelerometer_Breakout.kicad_pcb (KiCad board)
At the start: 2 copper layers, 13.5 x 13.5 mm, 5 parts, among them U1 H3LIS331DL, U2 4_Pin_header, U3 4_Pin_header

Commit message: Updated version (v3) with all the issues pointed out by Charles fixed
Parts:
- turned C1 to 270 degrees
Connections:
- net /CS renamed /H3LIS331DL_Accelerometer/CS_ACC
- net /INT_1 renamed /H3LIS331DL_Accelerometer/INT_1_ACC
- net /INT_2 renamed /H3LIS331DL_Accelerometer/INT_2_ACC
- net /SCL renamed /H3LIS331DL_Accelerometer/SCL_ACC
- net /SDA renamed /H3LIS331DL_Accelerometer/SDA_ACC
- net /SDO renamed /H3LIS331DL_Accelerometer/SDO_ACC
- C1 pad 1: GND -> +3V3
- C1 pad 2: +3V3 -> GND
Routing:
- net GND: track 25.3 -> 6.58 mm, vias 3 -> 2
- added copper zone on B.Cu, net GND
- added copper zone on F.Cu, net GND
