File: FHSD/Flash SD Board/Flash SD Board.kicad_pcb (KiCad board)
At the start: 2 copper layers, 27.9 x 20.7 mm, 5 parts

Commit message: Updated Flash SD Board Files
Refined Files
Parts:
-  : renamed from 9P
Routing:
- added copper zone on B.Cu, net GND
Other:
- board size 27.9 x 20.7 mm -> 27.9 x 25.8 mm
- board text added: "3v3"
- board text added: "CS_FL"
- board text added: "CS_SD"
- board text added: "GND"
- board text added: "HOLD"
- board text added: "MISO"
- board text added: "MOSI"
- board text added: "SCLK"
- board text added: "WP"
Changed lines of the file:
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@@
   (general
     (thickness 1.6)
-    (drawings 6)
+    (drawings 17)
     (tracks 64)
     (zones 0)
@@
   (page A4)
   (layers
-    (0 F.Cu signal)
-    (31 B.Cu signal)
+    (0 F.Cu signal hide)
+    (31 B.Cu signal hide)
     (32 B.Adhes user)
     (33 F.Adhes user)
@@
     (tags "microSD SD molex")
     (attr smd)
-    (fp_text reference "SD Connector" (at 0 -7.18) (layer F.SilkS)
+    (fp_text reference "SD Connector" (at 0 -7.6) (layer F.SilkS)
       (effects (font (size 1 1) (thickness 0.15)))
     )
@@
     (descr "Through hole straight pin header, 1x09, 2.54mm pitch, single row")
     (tags "Through hole pin header THT 1x09 2.54mm single row")
-    (fp_text reference 9P (at 0 -2.33 90) (layer F.SilkS)
+    (fp_text reference " " (at 0 -2.33 90) (layer F.SilkS)
       (effects (font (size 1 1) (thickness 0.15)))
     )
@@
     )
   )
-  (gr_text "Breakout Board" (at 144.1 111.7) (layer F.SilkS)
+  (gr_line (start 165.9 87) (end 138 87) (layer Edge.Cuts) (width 0.05))
+  (gr_line (start 165.9 92.1) (end 165.9 87) (layer Edge.Cuts) (width 0.05))
+  (gr_line (start 138 92.1) (end 138 87) (layer Edge.Cuts) (width 0.05))
+  (gr_text CS_FL (at 141.7 90.4 90) (layer F.SilkS)
+    (effects (font (size 1 1) (thickness 0.15)))
+  )
+  (gr_text WP (at 144.2 91.5 90) (layer F.SilkS)
+    (effects (font (size 1 1) (thickness 0.15)))
+  )
+  (gr_text HOLD (at 146.8 90.8 90) (layer F.SilkS)
+    (effects (font (size 1 1) (thickness 0.15)))
+  )
+  (gr_text SCLK (at 149.4 90.9 90) (layer F.SilkS)
+    (effects (font (size 1 1) (thickness 0.15)))
+  )
+  (gr_text MOSI (at 152 91 90) (layer F.SilkS)
+    (effects (font (size 1 1) (thickness 0.15)))
+  )
+  (gr_text MISO (at 154.5 91 90) (layer F.SilkS)
+    (effects (font (size 1 1) (thickness 0.15)))
+  )
+  (gr_text CS_SD (at 157 90.5 90) (layer F.SilkS)
+    (effects (font (size 1 1) (thickness 0.15)))
+  )
+  (gr_text GND (at 159.6 91.2 90) (layer F.SilkS)
+    (effects (font (size 1 1) (thickness 0.15)))
+  )
+  (gr_text 3v3 (at 162.2 91.3 90) (layer F.SilkS)
+    (effects (font (size 1 1) (thickness 0.15)))
+  )
+  (gr_text "Breakout Board" (at 144.2 111.7) (layer F.SilkS)
     (effects (font (size 1 1) (thickness 0.15)))
   )
   (gr_line (start 165.9 112.8) (end 138 112.8) (layer Edge.Cuts) (width 0.05))
-  (gr_text "SD & Flash" (at 144 110.1) (layer F.SilkS)
+  (gr_text "SD & Flash" (at 144.1 110.1) (layer F.SilkS)
     (effects (font (size 1 1) (thickness 0.15)))
   )
   (gr_line (start 138 92.1) (end 138 112.8) (layer Edge.Cuts) (width 0.05))
   (gr_line (start 165.9 92.1) (end 165.9 112.8) (layer Edge.Cuts) (width 0.05))
-  (gr_line (start 138 92.1) (end 165.9 92.1) (layer Edge.Cuts) (width 0.05))
   (via (at 156.2 107.8) (size 0.8) (drill 0.4) (layers F.Cu B.Cu) (net 1))
   (segment (start 156.238 106.161) (end 156.238 107.762) (width 0.25) (layer B.Cu) (net 1))
@@
       )
     )
+  )
+  (zone (net 4) (net_name GND) (layer B.Cu) (hatch edge 0.508)
+    (connect_pads (clearance 0.508))
+    (min_thickness 0.254)
+    (fill yes (arc_segments 32) (thermal_gap 0.508) (thermal_bridge_width 0.508))
+    (polygon
+      (pts
+        (xy 165.9 112.8) (xy 138 112.8) (xy 138 87) (xy 165.9 87)
+      )
+    )
+  )
+  (zone (net 4) (net_name GND) (layer F.Cu) (hatch edge 0.508)
+    (connect_pads (clearance 0.508))
+    (min_thickness 0.254)
+    (fill yes (arc_segments 32) (thermal_gap 0.508) (thermal_bridge_width 0.508))
+    (polygon
+      (pts
+        (xy 165.9 112.8) (xy 138 112.8) (xy 138 87.1) (xy 165.9 87)
+      )
+    )

Commit message: Fixed even more issues
Hopefully the last fixes
Parts:
- removed Flash Chip: W25N512GVPIT, Flash SD Board:W25N512GVPIT
- added U10: W25N512GVPIT, Footprint Library:W25N512GVPIT, F.Cu at (144.5, 102.4)
- J501: renamed from  
- Micro_SD301: renamed from SD Connector
- moved C401 0.06 mm to (143.8, 102.5), turned to 0 degrees
Connections:
- net /main/Flash Chip/CLK renamed /main/Flash Chip/SCLK
- C301 pad 1: +3V3 -> GND
- C301 pad 2: Net-(C301-Pad2) -> +3V3
- C401 pad 1: +3V3 -> GND
- C401 pad 2: Net-(C401-Pad2) -> +3V3
- Micro_SD301 pad 4: Net-(C301-Pad2) -> +3V3
Routing:
- net +3V3: track 24.9 -> 35.3 mm
- net /main/Flash Chip/MOSI: track 21.9 -> 27.6 mm
- net Net-(C401-Pad2): track 3.76 -> 0.00 mm, vias 1 -> 0
- net Net-(C301-Pad2): track 3.55 -> 0.00 mm, vias 1 -> 0
- net /main/Flash Chip/MISO: track 25.0 -> 27.7 mm, vias 3 -> 2

Commit message: Fixed tracing
Routing:
- net /main/Flash Chip/MOSI: track 27.6 -> 24.1 mm, vias 0 -> 1
