File: imu_hat/hat/hat.kicad_pcb (KiCad board)
At the start: 2 copper layers, 36.5 x 94 mm, 11 parts, among them J1 Conn_02x10_Odd_Even, U1 LSM9DS1

Commit message: Made New Dimensions
Parts:
- removed H2, H4: MountingHole, MountingHole:MountingHole_3mm
Other:
- board size 36.5 x 94 mm -> 36.5 x 35.5 mm
