File: Lambda Hat/LAMBDA HAT.sch (KiCad schematic (older format))
At the start: 8 parts, among them J1 Conn_02x10_Counter_Clockwise, U1 LAMBDA-9S-Global

Commit message: The hopefully fixed RF board from David
Parts:
- AE1: symbol Device:Antenna -> LAMBDA-HAT-rescue:Antenna-Device
- C1: symbol Device:C_Small -> LAMBDA-HAT-rescue:C_Small-Device
- H1, H2, H3, H4: symbol Mechanical:MountingHole -> LAMBDA-HAT-rescue:MountingHole-Mechanical
- J1: symbol Connector_Generic:Conn_02x10_Counter_Clockwise -> LAMBDA-HAT-rescue:Conn_02x10_Counter_Clockwise-Connector_Generic
Changed lines of the file:
@@
 $EndComp
 $Comp
-L power:+3.3V #PWR0101
+L LAMBDA-HAT-rescue:+3.3V-power #PWR0101
 U 1 1 5FF79490
 P 3250 4100
@@
 $EndComp
 $Comp
-L power:GND #PWR0102
+L LAMBDA-HAT-rescue:GND-power #PWR0102
 U 1 1 5FF7A1A0
 P 4100 4000
@@
 	4100 3900 3850 3900
 $Comp
-L Device:C_Small C1
+L LAMBDA-HAT-rescue:C_Small-Device C1
 U 1 1 5FF7DD84
 P 3450 3800
@@
 $EndComp
 $Comp
-L power:GND #PWR0104
+L LAMBDA-HAT-rescue:GND-power #PWR0104
 U 1 1 5FF7EBBB
 P 3450 3700
@@
 NoConn ~ 4100 4500
 $Comp
-L power:+3.3V #PWR0105
+L LAMBDA-HAT-rescue:+3.3V-power #PWR0105
 U 1 1 5FF8AAF4
 P 6650 4050
@@
 $EndComp
 $Comp
-L power:GND #PWR0106
+L LAMBDA-HAT-rescue:GND-power #PWR0106
 U 1 1 5FF8BF51
 P 6650 3850
@@
 Device active low\n
 $Comp
-L Device:Antenna AE1
+L LAMBDA-HAT-rescue:Antenna-Device AE1
 U 1 1 5FFA59EB
 P 3850 3400
@@
 $EndComp
 $Comp
-L Connector_Generic:Conn_02x10_Counter_Clockwise J1
+L LAMBDA-HAT-rescue:Conn_02x10_Counter_Clockwise-Connector_Generic J1
 U 1 1 5FFA9BC7
 P 6850 4250
@@
 NoConn ~ 6650 4750
 $Comp
-L Mechanical:MountingHole H1
+L LAMBDA-HAT-rescue:MountingHole-Mechanical H1
 U 1 1 5FFB1B80
 P 8550 4000
@@
 $EndComp
 $Comp
-L Mechanical:MountingHole H2
+L LAMBDA-HAT-rescue:MountingHole-Mechanical H2
 U 1 1 5FFB2BD8
 P 8550 4200
@@
 $EndComp
 $Comp
-L Mechanical:MountingHole H3
+L LAMBDA-HAT-rescue:MountingHole-Mechanical H3
 U 1 1 5FFB2DC8
 P 8550 4400
@@
 $EndComp
 $Comp
-L Mechanical:MountingHole H4
+L LAMBDA-HAT-rescue:MountingHole-Mechanical H4
 U 1 1 5FFB304B
 P 8550 4600

Commit message: Fixed global issues
Parts:
- AE1: symbol LAMBDA-HAT-rescue:Antenna-Device -> Device:Antenna
- C1: symbol LAMBDA-HAT-rescue:C_Small-Device -> Device:C
- H1, H2, H3, H4: symbol LAMBDA-HAT-rescue:MountingHole-Mechanical -> Mechanical:MountingHole
- J1: symbol LAMBDA-HAT-rescue:Conn_02x10_Counter_Clockwise-Connector_Generic -> Connector_Generic:Conn_02x10_Counter_Clockwise
- U1: symbol lambda-9s-global:LAMBDA-9S-Global -> lambda:LAMBDA-9S-Global
Connections:
- net labels added: +3V3
- net labels removed: +3.3V
- wire segments 5 -> 23
Changed lines of the file:
@@
 $EndDescr
 $Comp
-L lambda-9s-global:LAMBDA-9S-Global U1
+L lambda:LAMBDA-9S-Global U1
 U 1 1 5FF78303
 P 4500 3800
@@
 $EndComp
 $Comp
-L LAMBDA-HAT-rescue:+3.3V-power #PWR0101
+L power:+3V3 #PWR0101
 U 1 1 5FF79490
 P 3250 4100
 F 0 "#PWR0101" H 3250 3950 50  0001 C CNN
-F 1 "+3.3V" V 3265 4228 50  0000 L CNN
+F 1 "+3V3" V 3265 4228 50  0000 L CNN
 F 2 "" H 3250 4100 50  0001 C CNN
 F 3 "" H 3250 4100 50  0001 C CNN
@@
 $EndComp
 $Comp
-L LAMBDA-HAT-rescue:GND-power #PWR0102
+L power:GND #PWR0102
 U 1 1 5FF7A1A0
 P 4100 4000
@@
 	4100 3900 3850 3900
 $Comp
-L LAMBDA-HAT-rescue:C_Small-Device C1
+L Device:C C1
 U 1 1 5FF7DD84
-P 3450 3800
-F 0 "C1" H 3358 3754 50  0000 R CNN
-F 1 "100n" H 3358 3845 50  0000 R CNN
-F 2 "Capacitor_SMD:C_0603_1608Metric_Pad1.08x0.95mm_HandSolder" H 3450 3800 50  0001 C CNN
-F 3 "~" H 3450 3800 50  0001 C CNN
-	1    3450 3800
+P 3450 3750
+F 0 "C1" H 3358 3704 50  0000 R CNN
+F 1 "100n" H 3358 3795 50  0000 R CNN
+F 2 "Capacitor_SMD:C_0603_1608Metric_Pad1.08x0.95mm_HandSolder" H 3450 3750 50  0001 C CNN
+F 3 "~" H 3450 3750 50  0001 C CNN
+	1    3450 3750
 	-1   0    0    1
 $EndComp
 $Comp
-L LAMBDA-HAT-rescue:GND-power #PWR0104
+L power:GND #PWR0104
 U 1 1 5FF7EBBB
-P 3450 3700
-F 0 "#PWR0104" H 3450 3450 50  0001 C CNN
-F 1 "GND" H 3455 3527 50  0000 C CNN
-F 2 "" H 3450 3700 50  0001 C CNN
-F 3 "" H 3450 3700 50  0001 C CNN
-	1    3450 3700
+P 3450 3600
+F 0 "#PWR0104" H 3450 3350 50  0001 C CNN
+F 1 "GND" H 3455 3427 50  0000 C CNN
+F 2 "" H 3450 3600 50  0001 C CNN
+F 3 "" H 3450 3600 50  0001 C CNN
+	1    3450 3600
 	-1   0    0    1
 $EndComp
@@
 NoConn ~ 4100 4500
 $Comp
-L LAMBDA-HAT-rescue:+3.3V-power #PWR0105
+L power:+3V3 #PWR0105
 U 1 1 5FF8AAF4
-P 6650 4050
-F 0 "#PWR0105" H 6650 3900 50  0001 C CNN
-F 1 "+3.3V" V 6665 4178 50  0000 L CNN
-F 2 "" H 6650 4050 50  0001 C CNN
-F 3 "" H 6650 4050 50  0001 C CNN
-	1    6650 4050
+P 6600 4050
+F 0 "#PWR0105" H 6600 3900 50  0001 C CNN
+F 1 "+3V3" V 6615 4178 50  0000 L CNN
+F 2 "" H 6600 4050 50  0001 C CNN
+F 3 "" H 6600 4050 50  0001 C CNN
+	1    6600 4050
 	0    -1   -1   0
 $EndComp
 $Comp
-L LAMBDA-HAT-rescue:GND-power #PWR0106
+L power:GND #PWR0106
 U 1 1 5FF8BF51
-P 6650 3850
-F 0 "#PWR0106" H 6650 3600 50  0001 C CNN
-F 1 "GND" V 6655 3722 50  0000 R CNN
-F 2 "" H 6650 3850 50  0001 C CNN
-F 3 "" H 6650 3850 50  0001 C CNN
-	1    6650 3850
+P 6600 3850
+F 0 "#PWR0106" H 6600 3600 50  0001 C CNN
+F 1 "GND" V 6605 3722 50  0000 R CNN
+F 2 "" H 6600 3850 50  0001 C CNN
+F 3 "" H 6600 3850 50  0001 C CNN
+	1    6600 3850
 	0    1    1    0
 $EndComp
@@
 Device active low\n
 $Comp
-L LAMBDA-HAT-rescue:Antenna-Device AE1
+L Device:Antenna AE1
 U 1 1 5FFA59EB
 P 3850 3400
@@
 $EndComp
 $Comp
-L LAMBDA-HAT-rescue:Conn_02x10_Counter_Clockwise-Connector_Generic J1
+L Connector_Generic:Conn_02x10_Counter_Clockwise J1
 U 1 1 5FFA9BC7
 P 6850 4250
@@
 NoConn ~ 6650 4750
 $Comp
-L LAMBDA-HAT-rescue:MountingHole-Mechanical H1
+L Mechanical:MountingHole H1
 U 1 1 5FFB1B80
 P 8550 4000
@@
 $EndComp
 $Comp
-L LAMBDA-HAT-rescue:MountingHole-Mechanical H2
+L Mechanical:MountingHole H2
 U 1 1 5FFB2BD8
 P 8550 4200
@@
 $EndComp
 $Comp
-L LAMBDA-HAT-rescue:MountingHole-Mechanical H3
+L Mechanical:MountingHole H3
 U 1 1 5FFB2DC8
 P 8550 4400
@@
 $EndComp
 $Comp
-L LAMBDA-HAT-rescue:MountingHole-Mechanical H4
+L Mechanical:MountingHole H4
 U 1 1 5FFB304B
 P 8550 4600
@@
 Wire Wire Line
 	3850 3900 3850 3600
-Text HLabel 5100 3900 2    50   Input ~ 0
+Text HLabel 5150 3900 2    50   Input ~ 0
 nCS
-Text HLabel 5100 4000 2    50   Input ~ 0
+Text HLabel 5150 4000 2    50   Input ~ 0
 MOSI
-Text HLabel 5100 4100 2    50   Input ~ 0
+Text HLabel 5150 4100 2    50   Input ~ 0
 MISO
-Text HLabel 5100 4200 2    50   Input ~ 0
+Text HLabel 5150 4200 2    50   Input ~ 0
 SCK
-Text HLabel 5100 4300 2    50   Input ~ 0
+Text HLabel 5150 4300 2    50   Input ~ 0
 RESET
-Text HLabel 4100 4200 0    50   Input ~ 0
+Text HLabel 4050 4200 0    50   Input ~ 0
 RX_SWITCH
-Text HLabel 4100 4300 0    50   Input ~ 0
+Text HLabel 4050 4300 0    50   Input ~ 0
 TX_SWITCH
-Text HLabel 4100 4400 0    50   Input ~ 0
+Text HLabel 4050 4400 0    50   Input ~ 0
 DIO
-Text HLabel 7150 4350 2    50   Input ~ 0
+Text HLabel 7200 4350 2    50   Input ~ 0
 nCS
-Text HLabel 7150 4250 2    50   Input ~ 0
+Text HLabel 7200 4250 2    50   Input ~ 0
 MOSI
-Text HLabel 7150 4050 2    50   Input ~ 0
+Text HLabel 7200 4050 2    50   Input ~ 0
 MISO
-Text HLabel 7150 4450 2    50   Input ~ 0
+Text HLabel 7200 4450 2    50   Input ~ 0
 RESET
-Text HLabel 7150 4150 2    50   Input ~ 0
+Text HLabel 7200 4150 2    50   Input ~ 0
 SCK
-Text HLabel 7150 4750 2    50   Input ~ 0
+Text HLabel 7200 4750 2    50   Input ~ 0
 DIO
-Text HLabel 7150 4650 2    50   Input ~ 0
+Text HLabel 7200 4650 2    50   Input ~ 0
 TX_SWITCH
-Text HLabel 7150 4550 2    50   Input ~ 0
+Text HLabel 7200 4550 2    50   Input ~ 0
 RX_SWITCH
+Wire Wire Line
+	6600 3850 6650 3850
+Wire Wire Line
+	6650 4050 6600 4050
+Wire Wire Line
+	5100 3900 5150 3900
+Wire Wire Line
+	5150 4000 5100 4000
+Wire Wire Line
+	5100 4100 5150 4100
+Wire Wire Line
+	5150 4200 5100 4200
+Wire Wire Line
+	5100 4300 5150 4300
+Wire Wire Line
+	4100 4200 4050 4200
+Wire Wire Line
+	4050 4300 4100 4300
+Wire Wire Line
+	4100 4400 4050 4400
+Wire Wire Line
+	7150 4050 7200 4050
+Wire Wire Line
+	7150 4150 7200 4150
+Wire Wire Line
+	7150 4250 7200 4250
+Wire Wire Line
+	7150 4350 7200 4350
+Wire Wire Line
+	7150 4450 7200 4450
+Wire Wire Line
+	7150 4550 7200 4550
+Wire Wire Line
+	7150 4650 7200 4650
+Wire Wire Line
+	7150 4750 7200 4750
 $EndSCHEMATC

Commit message: Possibly Fixed Footprint Issue
Parts:
- U1: symbol lambda:LAMBDA-9S-Global -> lambda-9s-global:LAMBDA-9S-Global
Changed lines of the file:
@@
 $EndDescr
 $Comp
-L lambda:LAMBDA-9S-Global U1
+L lambda-9s-global:LAMBDA-9S-Global U1
 U 1 1 5FF78303
 P 4500 3800
