File: GPS&RF/GPS&RF/GPS.sch (KiCad schematic (older format))
At the start: 11 parts, among them IC1 FGPMMOPA6H, J1 U.FL-R-SMT(10)

Commit message: Finished the GPS&RF schematic
Replaced the 8 pin conn with a 13 pin conn_molex_PicoBlade
Parts:
- removed R2, R3: 330ohm, Resistor_SMD:R_0603_1608Metric_Pad1.05x0.95mm_HandSolder, symbol Device:R_US
- BT1: symbol 120591-1:120591-1 -> GPS&RF-rescue:120591-1-120591-1
- IC1: symbol FGPMMOPA6H:FGPMMOPA6H -> GPS&RF-rescue:FGPMMOPA6H-FGPMMOPA6H
- J1: symbol U.FL-R-SMT_10_:U.FL-R-SMT(10) -> GPS&RF-rescue:U.FL-R-SMT(10)-U.FL-R-SMT_10_
Connections:
- no-connect marks 8 -> 10
Changed lines of the file:
@@
 $EndDescr
 $Comp
-L FGPMMOPA6H:FGPMMOPA6H IC1
+L GPS&RF-rescue:FGPMMOPA6H-FGPMMOPA6H IC1
 U 1 1 6063EB03
 P 4970 4000
@@
 	3580 4300 3580 4550
 $Comp
-L 120591-1:120591-1 BT1
+L GPS&RF-rescue:120591-1-120591-1 BT1
 U 1 1 60647D28
 P 3580 4750
+AR Path="/60647D28" Ref="BT1"  Part="1"
+AR Path="/60625D95/60647D28" Ref="BT1"  Part="1"
 F 0 "BT1" V 3440 4560 50  0000 L CNN
 F 1 "BATT" V 3740 4530 50  0000 L CNN
@@
 Wire Wire Line
 	4970 4700 4770 4700
-$Comp
-L power:GND #PWR0110
-U 1 1 6064CCAC
-P 4770 4700
-F 0 "#PWR0110" H 4770 4450 50  0001 C CNN
-F 1 "GND" V 4680 4730 50  0000 R CNN
-F 2 "" H 4770 4700 50  0001 C CNN
-F 3 "" H 4770 4700 50  0001 C CNN
-	1    4770 4700
-	0    1    1    0
-$EndComp
-$Comp
-L power:PWR_FLAG #FLG0101
-U 1 1 6064D61B
-P 4970 4700
-F 0 "#FLG0101" H 4970 4775 50  0001 C CNN
-F 1 "PWR_FLAG" V 4910 4550 50  0000 L CNN
-F 2 "" H 4970 4700 50  0001 C CNN
-F 3 "~" H 4970 4700 50  0001 C CNN
-	1    4970 4700
-	0    -1   -1   0
-$EndComp
-Connection ~ 4970 4700
-Wire Wire Line
-	4380 4800 4490 4800
-Wire Wire Line
-	4380 4900 4600 4900
-$Comp
-L Device:R_US R2
-U 1 1 60650174
-P 4640 4800
-F 0 "R2" V 4580 4680 50  0000 C CNN
-F 1 "330ohm" V 4700 4800 50  0000 C CNN
-F 2 "Resistor_SMD:R_0603_1608Metric_Pad1.05x0.95mm_HandSolder" V 4680 4790 50  0001 C CNN
-F 3 "~" H 4640 4800 50  0001 C CNN
-	1    4640 4800
-	0    1    1    0
-$EndComp
-Wire Wire Line
-	4790 4800 4970 4800
-Wire Wire Line
-	4900 4900 4970 4900
-Text HLabel 4380 4800 0    50   Input ~ 0
-TX
-Text HLabel 4380 4900 0    50   Input ~ 0
-RX
-$Comp
-L Device:R_US R3
-U 1 1 60651105
-P 4750 4900
-F 0 "R3" V 4710 5020 50  0000 C CNN
-F 1 "330ohm" V 4830 4920 50  0000 C CNN
-F 2 "Resistor_SMD:R_0603_1608Metric_Pad1.05x0.95mm_HandSolder" V 4790 4890 50  0001 C CNN
-F 3 "~" H 4750 4900 50  0001 C CNN
-	1    4750 4900
-	0    1    1    0
-$EndComp
 Wire Wire Line
 	6370 4100 6510 4100
@@
 Connection ~ 6840 4900
 $Comp
-L U.FL-R-SMT_10_:U.FL-R-SMT(10) J1
+L GPS&RF-rescue:U.FL-R-SMT(10)-U.FL-R-SMT_10_ J1
 U 1 1 60658D1A
 P 7120 4900
@@
 	-1   0    0    1
 $EndComp
+Connection ~ 4970 4700
+$Comp
+L power:PWR_FLAG #FLG0101
+U 1 1 6064D61B
+P 4970 4700
+F 0 "#FLG0101" H 4970 4775 50  0001 C CNN
+F 1 "PWR_FLAG" V 4900 4620 50  0000 L CNN
+F 2 "" H 4970 4700 50  0001 C CNN
+F 3 "~" H 4970 4700 50  0001 C CNN
+	1    4970 4700
+	0    -1   -1   0
+$EndComp
+$Comp
+L power:GND #PWR0110
+U 1 1 6064CCAC
+P 4770 4700
+F 0 "#PWR0110" H 4770 4450 50  0001 C CNN
+F 1 "GND" V 4680 4730 50  0000 R CNN
+F 2 "" H 4770 4700 50  0001 C CNN
+F 3 "" H 4770 4700 50  0001 C CNN
+	1    4770 4700
+	0    1    1    0
+$EndComp
+NoConn ~ 4970 4800
+NoConn ~ 4970 4900
 $EndSCHEMATC

Commit message: Finished SCH and PCB
Finished everything, might need to edit a few things but pushing the 'final' now
Parts:
- C2, C3, C4: footprint Capacitor_SMD:C_0603_1608Metric_Pad1.05x0.95mm_HandSolder -> Capacitor_SMD:C_0603_1608Metric_Pad1.08x0.95mm_HandSolder
- R1: footprint Resistor_SMD:R_0603_1608Metric_Pad1.05x0.95mm_HandSolder -> Resistor_SMD:R_0603_1608Metric_Pad0.98x0.95mm_HandSolder
Connections:
- net RX_D2: now reaches IC1.10 (RX)
- net TX_D2: now reaches IC1.9 (TX)
- no-connect marks 10 -> 8
Changed lines of the file:
@@
 F 0 "C3" H 4450 3840 50  0000 L CNN
 F 1 "1uF" H 4450 3680 50  0000 L CNN
-F 2 "Capacitor_SMD:C_0603_1608Metric_Pad1.05x0.95mm_HandSolder" H 4458 3610 50  0001 C CNN
+F 2 "Capacitor_SMD:C_0603_1608Metric_Pad1.08x0.95mm_HandSolder" H 4458 3610 50  0001 C CNN
 F 3 "~" H 4420 3760 50  0001 C CNN
 	1    4420 3760
@@
 F 0 "C4" H 4720 3840 50  0000 L CNN
 F 1 "0.01uF" H 4720 3680 50  0000 L CNN
-F 2 "Capacitor_SMD:C_0603_1608Metric_Pad1.05x0.95mm_HandSolder" H 4718 3610 50  0001 C CNN
+F 2 "Capacitor_SMD:C_0603_1608Metric_Pad1.08x0.95mm_HandSolder" H 4718 3610 50  0001 C CNN
 F 3 "~" H 4680 3760 50  0001 C CNN
 	1    4680 3760
@@
 F 0 "C2" H 3820 4620 50  0000 L CNN
 F 1 "1uF" H 3820 4460 50  0000 L CNN
-F 2 "Capacitor_SMD:C_0603_1608Metric_Pad1.05x0.95mm_HandSolder" H 3828 4390 50  0001 C CNN
+F 2 "Capacitor_SMD:C_0603_1608Metric_Pad1.08x0.95mm_HandSolder" H 3828 4390 50  0001 C CNN
 F 3 "~" H 3790 4540 50  0001 C CNN
 	1    3790 4540
@@
 F 0 "R1" V 4500 4520 50  0000 C CNN
 F 1 "330ohm" V 4630 4400 50  0000 C CNN
-F 2 "Resistor_SMD:R_0603_1608Metric_Pad1.05x0.95mm_HandSolder" V 4580 4390 50  0001 C CNN
+F 2 "Resistor_SMD:R_0603_1608Metric_Pad0.98x0.95mm_HandSolder" V 4580 4390 50  0001 C CNN
 F 3 "~" H 4540 4400 50  0001 C CNN
 	1    4540 4400
@@
 	0    1    1    0
 $EndComp
-NoConn ~ 4970 4800
-NoConn ~ 4970 4900
+Wire Wire Line
+	4970 4800 4600 4800
+Wire Wire Line
+	4970 4900 4600 4900
+Text HLabel 4600 4800 0    50   Input ~ 0
+TX_D2
+Text HLabel 4600 4900 0    50   Input ~ 0
+RX_D2
 $EndSCHEMATC
