File: GPS&RF/GPS&RF/RF.sch (KiCad schematic (older format))
At the start: 3 parts, among them U1 LAMBDA-9S-Global

Commit message: Finished the GPS&RF schematic
Replaced the 8 pin conn with a 13 pin conn_molex_PicoBlade
Parts:
- U1: symbol lambda-9s-global:LAMBDA-9S-Global -> GPS&RF-rescue:LAMBDA-9S-Global-lambda-9s-global
Connections:
- net DIO: no longer names the net of U1.6 (DIO0)
- no-connect marks 5 -> 6
Changed lines of the file:
@@
 $EndDescr
 $Comp
-L lambda-9s-global:LAMBDA-9S-Global U1
+L GPS&RF-rescue:LAMBDA-9S-Global-lambda-9s-global U1
 U 1 1 606260CA
 P 5030 3580
+AR Path="/60625EDB/606260CA" Ref="U1"  Part="1"
+AR Path="/606260CA" Ref="U1"  Part="1"
 F 0 "U1" H 5130 3705 50  0000 C CNN
 F 1 "LAMBDA-9S-Global" H 5130 3614 50  0000 C CNN
@@
 Wire Wire Line
 	4630 4080 4450 4080
-Wire Wire Line
-	4630 4180 4450 4180
 Wire Wire Line
 	5810 4080 5630 4080
@@
 Text HLabel 4450 4080 0    50   Input ~ 0
 TX
-Text HLabel 4450 4180 0    50   Input ~ 0
-DIO
 Text HLabel 5810 3680 2    50   Input ~ 0
 CS
@@
 Text Notes 6370 3630 2    50   ~ 0
 DEVICE ACTIVE LOW
+NoConn ~ 4630 4180
 $EndSCHEMATC

Commit message: Finished SCH and PCB
Finished everything, might need to edit a few things but pushing the 'final' now
Parts:
- C1: footprint Capacitor_SMD:C_0603_1608Metric_Pad1.05x0.95mm_HandSolder -> Capacitor_SMD:C_0603_1608Metric_Pad1.08x0.95mm_HandSolder
Connections:
- net RX renamed RX_D1
- net TX renamed TX_D1
Changed lines of the file:
@@
 F 0 "C1" H 4195 3516 50  0000 L CNN
 F 1 "100nF" H 4110 3380 50  0000 L CNN
-F 2 "Capacitor_SMD:C_0603_1608Metric_Pad1.05x0.95mm_HandSolder" H 4118 3320 50  0001 C CNN
+F 2 "Capacitor_SMD:C_0603_1608Metric_Pad1.08x0.95mm_HandSolder" H 4118 3320 50  0001 C CNN
 F 3 "~" H 4080 3470 50  0001 C CNN
 	1    4080 3470
@@
 	4080 3140 4080 3320
 Text HLabel 4450 3980 0    50   Input ~ 0
-RX
+RX_D1
 Text HLabel 4450 4080 0    50   Input ~ 0
-TX
+TX_D1
 Text HLabel 5810 3680 2    50   Input ~ 0
 CS
